Commit message: modified waypoints, nav2, and racecar urdf model

File: src/auna_gazebo/models/race_car/model.urdf (robot description, URDF)
Before this commit: robot sam_bot, 6 links, 5 joints
Joints:
- joint base_link_joint: origin xyz=${-base_x_origin_to_wheel_origin} 0 0.05 rpy=0 0 0 -> xyz=${base_x_origin_to_wheel_origin} 0 0.05 rpy=0 0 0
