Commit message: Add GPS link and sensor to race car model; define properties and Gazebo plugin for GPS functionality

File: packages/src/auna_gazebo/models/race_car/model.urdf (robot description, URDF)
Before this commit: robot sam_bot, 6 links, 5 joints
Links:
- added link $(arg namespace)gps_link, mass ${gpsMass}; collision box size=${gpsSizeL} ${gpsSizeB} ${gpsSizeH}; visual box size=${gpsSizeL} ${gpsSizeB} ${gpsSizeH}
Joints:
- added joint gps_joint: type fixed, parent $(arg namespace)chassis, child $(arg namespace)gps_link, origin xyz=-0.1 0 0.15 rpy=0 0 0

Commit message: Refactor command velocity topics and implement RViz panels
- Changed the command velocity topic from "cmd_vel" to "cmd_vel_cacc" in CACC controller.
- Updated the bringup launch file to separate SLAM, Localization, and Navigation commands.
- Modified the URDF model to remove unnecessary namespace arguments for links and joints.
- Created a new CmdVelMuxPanel for selecting command velocity sources (CACC, Teleop, Nav2) in RViz.
- Implemented a GlobalEmergencyStopPanel to send emergency stop commands to multiple namespaces.
- Updated CMakeLists.txt to include necessary Qt dependencies and removed unused std_srvs dependency.
- Adjusted package.xml to reflect the removal of std_srvs and added geometry_msgs dependency.
- Updated plugins_description.xml to register new RViz panels.
- Changed teleoperation topic names to "cmd_vel_teleop" for consistency across the system.

File: packages/src/auna_gazebo/models/race_car/model.urdf (robot description, URDF)
Before this commit: robot sam_bot, 7 links, 6 joints
Links:
- removed link $(arg namespace)base_link
- removed link $(arg namespace)camera
- removed link $(arg namespace)chassis
- removed link $(arg namespace)gps_link
- removed link $(arg namespace)imu_link
- removed link $(arg namespace)laser
- removed link $(arg namespace)steering_wheel
- added link base_link
- added link camera, mass ${cameraMass}; collision box size=${cameraSizeL} ${cameraSizeH} ${cameraSizeB}; visual mesh filename=file:///$(find auna_gazebo)/models/race_car/meshes/ZED.dae
- added link chassis, mass ${bodyMass}; collision box size=${bodySizeL} ${bodySizeB} ${bodySizeH}; visual mesh filename=file:///$(find auna_gazebo)/models/race_car/meshes/car.dae
- added link gps_link, mass ${gpsMass}; collision box size=${gpsSizeL} ${gpsSizeB} ${gpsSizeH}; visual box size=${gpsSizeL} ${gpsSizeB} ${gpsSizeH}
- added link imu_link
- added link laser, mass ${hokuyoMass}; collision box size=${hokuyoSize} ${hokuyoSize} ${hokuyoSize}; visual mesh filename=file:///$(find auna_gazebo)/models/race_car/meshes/hokuyo.d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
- added link steering_wheel, mass 0.1; collision box size=0.01 0.01 0.01; visual box size=0.01 0.01 0.01
Joints:
- joint base_link_joint: child $(arg namespace)chassis -> chassis; parent $(arg namespace)base_link -> base_link
- joint camera_joint: child $(arg namespace)camera -> camera; parent $(arg namespace)chassis -> chassis
- joint gps_joint: child $(arg namespace)gps_link -> gps_link; parent $(arg namespace)chassis -> chassis
- joint imu_joint: child $(arg namespace)imu_link -> imu_link; parent $(arg namespace)chassis -> chassis
- joint laser_joint: child $(arg namespace)laser -> laser; parent $(arg namespace)chassis -> chassis
- joint steering_wheel_joint: child $(arg namespace)steering_wheel -> steering_wheel; parent $(arg namespace)chassis -> chassis

Commit message: Update EKF configuration and refine IMU sensor settings for improved performance

File: packages/src/auna_gazebo/models/race_car/model.urdf (robot description, URDF)
Before this commit: robot sam_bot, 7 links, 6 joints
Links:
- link imu_link: mass None -> 0.01
